File: tests/fixtures/Arduino_Mega/Arduino_Mega.kicad_sch (KiCad schematic)
At the start: 11 parts, among them J1 Power, J2 PWM, J3 Analog, J4 PWM, J5 Analog, J6 Communication, J7 Digital

Commit message: feat(09): add GRPO spatial reasoning training pipeline (Phase 9)
Phase 9: DeepSeek-style RL training with coordinate-grounded reward
signals on synthetic PCB maze data. 90 new tests passing.

Plans executed:
- 09-01: Synthetic data pipeline (MazeSample, MazeDataset, parallel gen)
- 09-02: Cold-start reasoning chain synthesis (DFS exploration, JSONL)
- 09-03: Reward model (per-step dense rewards, anti-hacking, neural model)
- 09-04: GRPO training loop, evaluation harness, single-command pipeline

New modules: training/{dataset,generator,chains,chain_builder,
chain_writer,reward,reward_hacking,reward_model,grpo,evaluation,pipeline}

Generated with [Claude Code](https://claude.ai/code)
via [Happy](https://happy.engineering)

Co-Authored-By: Claude <noreply@anthropic.com>
Co-Authored-By: Happy <yesreply@happy.engineering>
Parts:
- added R?: (no value), symbol Device:R_Small_US
Changed lines of the file:
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@@
+    )
+  )
+  (symbol (lib_name "Device:R_Small_US") (lib_id "Device:R_Small_US") (at 50 30)
+    (in_bom yes) (on_board yes)
+    (property "Reference" "R?" (id 0) (at 0 0)
+      (effects (font (size 1.27 1.27)))
+    )
+    (property "Value" "" (id 1) (at 0 0)
+      (effects (font (size 1.27 1.27)))
+    )
+    (property "Footprint" "" (id 2) (at 0 0)
+      (effects (font (size 1.27 1.27)) hide)
+    )
+    (property "Datasheet" "~" (id 3) (at 0 0)
+      (effects (font (size 1.27 1.27)) hide)
     )
   )
