File: tests/fixtures/Arduino_Mega/Arduino_Mega.kicad_sch (KiCad schematic)
At the start: 13 parts, among them J1 Power, J2 PWM, J3 Analog, J4 PWM, J5 Analog, J6 Communication, J7 Digital

Commit message: feat: fine-tuned PCB reasoning model + HF Hub + local inference
SFT + GRPO LoRA training on Qwen2.5-0.5B-Instruct (7,441 samples,
loss 2.20->0.69 SFT, 0.46->0.28 GRPO). Added LocalLLMClient with
HF Hub auto-download fallback, `kicad-agent analyze` CLI command,
model evaluation framework, schematic graph builder, EasyEDA API
integration, and 100K crawl discovery pipeline.

Model hosted at: bretbouchard/kicad-agent-pcb-adapter

Generated with [Claude Code](https://claude.ai/code)
via [Happy](https://happy.engineering)

Co-Authored-By: Claude <noreply@anthropic.com>
Co-Authored-By: Happy <yesreply@happy.engineering>
Parts:
- added R? (x27): (no value), symbol Device:R_Small_US
